File: isp32/panel.kicad_pcb (KiCad board)
At the start: 2 copper layers, 73 x 102 mm, 250 parts, among them J1 BAT1, J10 LoRa_ANT, J12 Micro_SD_Card, J2 Switching, J3 USB_C_Receptacle_USB2.0, J4 ADC, J5 GPS_ANT, J6 F0, J7 F1, J8 BUZZ, J9 ANT, M1 Motor_Servo, M2 Motor_Servo, M3 Motor_Servo, M4 Motor_Servo, Q1 BSS138, Q2 S8050, Q3 IRLML6402, Q4 BSS138, Q5 IRLML6402, Q6 IRLML6402, Q7 IRLML6402, Q8 BSS138, Q9 BSS138, SW1 RST, U1 AZ1117-3.3, U10 BMP280, U11 MPU-9250, U2 MP2315, U3 STM32G030F6, U4 AZ1117-1.8, U6 24LC32, U7 NEO-XM, U8 ESP32-S3-WROOM-1U, U9 RFM98W-315S2

Commit message: feat: isp32 2023 12 19
Parts:
- removed the C1 at (103.2, 109.6)
- removed the C1 at (103.2, 61.6)
- removed C17 (x2): 22u, Capacitor_SMD:C_0603_1608Metric
- removed the C2 at (94.2, 99.9)
- removed the C2 at (94.2, 51.9)
- removed the C4 at (97.6, 54.3)
- removed the C4 at (97.6, 102.3)
- removed the C5 at (96.2, 61.8)
- removed the C5 at (96.2, 109.8)
- removed the C7 at (102.4, 105.5)
- removed the C7 at (102.4, 57.5)
- removed the C8 at (97.7, 52.0)
- removed the C8 at (97.7, 100.0)
- removed the D1 at (98.0, 66.0)
- removed the D1 at (98.0, 114.0)
- removed the D6 at (92.8, 63.6)
- removed the D6 at (92.8, 111.6)
- removed the L3 at (93.2, 104.7)
- removed the L3 at (93.2, 56.7)
- removed Q7 (x2): IRLML6402, Package_TO_SOT_SMD:SOT-23
- removed the R10 at (101.5, 61.6)
- removed the R10 at (101.5, 109.6)
- removed the R11 at (102.4, 59.1)
- removed the R11 at (102.4, 107.1)
- removed the R21 at (102.1, 55.9)
- removed the R21 at (102.1, 103.9)
- removed R27 (x2): 100k, Resistor_SMD:R_0603_1608Metric
- removed the R3 at (98.0, 61.6)
- removed the R3 at (98.0, 109.6)
- removed the R8 at (100.7, 54.4)
- removed the R8 at (100.7, 102.4)
- removed the R9 at (99.8, 109.6)
- removed the R9 at (99.8, 61.6)
- removed the REF** at (95.1, 96.4)
- removed the REF** at (95.1, 48.4)
- removed the REF** at (112.1, 90.2)
- removed the REF** at (118.1, 42.3)
- removed the REF** at (118.1, 90.3)
- removed the REF** at (112.1, 42.2)
- removed the TP1 at (108.2, 30.8)
- removed the TP1 at (108.2, 78.8)
- removed the TP3 at (108.2, 29.5)
- removed the TP3 at (108.2, 77.5)
- removed the TP4 at (108.2, 28.2)
- removed the TP4 at (108.2, 76.2)
- removed the TP5 at (108.2, 75.0)
- removed the TP5 at (108.2, 27.0)
- removed the U1 at (102.6, 101.6)
- removed the U1 at (102.6, 53.6)
- removed the U2 at (98.3, 57.8)
- removed the U2 at (98.3, 105.8)
- removed the kibuzzard-63CD1E61 at (110.1, 30.8)
- removed the kibuzzard-63CD1E61 at (110.1, 78.8)
- removed the kibuzzard-63CD1E7F at (110.1, 26.9)
- removed the kibuzzard-63CD1E7F at (110.1, 74.9)
- removed the kibuzzard-63CD1EC0 at (110.1, 28.2)
- removed the kibuzzard-63CD1EC0 at (110.1, 76.2)
- removed the kibuzzard-63CD1EC5 at (110.1, 77.5)
- removed the kibuzzard-63CD1EC5 at (110.1, 29.5)
- added C1: 22u, Capacitor_SMD:C_0603_1608Metric, B.Cu at (105.2, 114.9)
- added C1: 22u, Capacitor_SMD:C_0603_1608Metric, B.Cu at (105.2, 64.9)
- added C2: 220u, Capacitor_Tantalum_SMD:CP_EIA-3528-12_Kemet-T, B.Cu at (92.4, 102.8)
- added C2: 220u, Capacitor_Tantalum_SMD:CP_EIA-3528-12_Kemet-T, B.Cu at (92.4, 52.8)
- added C4: 100n, Capacitor_SMD:C_0603_1608Metric, B.Cu at (96.8, 110.9)
- added C4: 100n, Capacitor_SMD:C_0603_1608Metric, B.Cu at (96.8, 60.9)
- added C5: 100n, Capacitor_SMD:C_0805_2012Metric, B.Cu at (95.9, 107.0)
- added C5: 100n, Capacitor_SMD:C_0805_2012Metric, B.Cu at (95.9, 57.0)
- added C7: NC, Capacitor_SMD:C_0603_1608Metric, B.Cu at (95.9, 100.2)
- added C7: NC, Capacitor_SMD:C_0603_1608Metric, B.Cu at (95.9, 50.2)
- added C8: 22u, Capacitor_SMD:C_0603_1608Metric, B.Cu at (105.2, 116.5)
- added C8: 22u, Capacitor_SMD:C_0603_1608Metric, B.Cu at (105.2, 66.5)
- added D1: Zener, Diode_SMD:D_SOD-123, B.Cu at (96.2, 114.9)
- added D1: Zener, Diode_SMD:D_SOD-123, B.Cu at (96.2, 64.9)
- added D6: TVS, Diode_SMD:D_SMB, B.Cu at (92.6, 113.6)
- added D6: TVS, Diode_SMD:D_SMB, B.Cu at (92.6, 63.6)
- added D8: D_Shockley, Diode_SMD:D_SOD-123, F.Cu at (102.4, 110.1)
- added D8: D_Shockley, Diode_SMD:D_SOD-123, F.Cu at (102.4, 60.1)
- added J11: Power Modules, Connector_PinSocket_2.54mm:PinSocket_1x04_P2.54mm_Vertical, F.Cu at (80.5, 59.1)
- added J11: Power Modules, Connector_PinSocket_2.54mm:PinSocket_1x04_P2.54mm_Vertical, F.Cu at (80.5, 109.1)
- added L3: 5.5, Inductor_SMD:L_Sunlord_SWPA5020S, B.Cu at (100.8, 114.8)
- added L3: 5.5, Inductor_SMD:L_Sunlord_SWPA5020S, B.Cu at (100.8, 64.8)
- added R10: 7k5, Resistor_SMD:R_0603_1608Metric, B.Cu at (95.1, 104.2)
- added R10: 7k5, Resistor_SMD:R_0603_1608Metric, B.Cu at (95.1, 54.2)
- added R11: 40.2k, Resistor_SMD:R_0603_1608Metric, B.Cu at (95.9, 51.8)
- added R11: 40.2k, Resistor_SMD:R_0603_1608Metric, B.Cu at (95.9, 101.8)
- added R21: 75k, Resistor_SMD:R_0603_1608Metric, B.Cu at (100.5, 53.8)
- added R21: 75k, Resistor_SMD:R_0603_1608Metric, B.Cu at (100.5, 103.8)
- added R3: 100k, Resistor_SMD:R_0603_1608Metric, B.Cu at (93.1, 57.4)
- added R3: 100k, Resistor_SMD:R_0603_1608Metric, B.Cu at (93.1, 107.4)
- added R8: 20, Resistor_SMD:R_0603_1608Metric, B.Cu at (96.8, 109.3)
- added R8: 20, Resistor_SMD:R_0603_1608Metric, B.Cu at (96.8, 59.3)
- added R9: 20k, Resistor_SMD:R_0603_1608Metric, B.Cu at (96.7, 54.1)
- added R9: 20k, Resistor_SMD:R_0603_1608Metric, B.Cu at (96.7, 104.1)
- added REF**: NPTH, NPTH, F.Cu at (91.2, 68.5)
- added REF**: NPTH, NPTH, F.Cu at (78.0, 43.2)
- added REF**: NPTH, NPTH, F.Cu at (78.0, 59.3)
- added REF**: NPTH, NPTH, F.Cu at (78.0, 74.6)
- added REF**: NPTH, NPTH, F.Cu at (111.5, 69.5)
- added REF**: NPTH, NPTH, F.Cu at (128.5, 68.5)
- added REF**: NPTH, NPTH, F.Cu at (127.7, 69.5)
- added REF**: NPTH, NPTH, F.Cu at (132.0, 41.6)
- added REF**: NPTH, NPTH, F.Cu at (78.0, 27.8)
- added REF**: NPTH, NPTH, F.Cu at (78.0, 89.2)
- added REF**: NPTH, NPTH, F.Cu at (97.7, 68.5)
- added REF**: NPTH, NPTH, F.Cu at (78.0, 88.3)
- added REF**: NPTH, NPTH, F.Cu at (78.0, 56.9)
- added REF**: NPTH, NPTH, F.Cu at (78.0, 102.1)
- added REF**: NPTH, NPTH, F.Cu at (132.0, 86.7)
- added REF**: NPTH, NPTH, F.Cu at (122.0, 69.5)
- added REF**: NPTH, NPTH, F.Cu at (132.0, 102.9)
- added REF**: NPTH, NPTH, F.Cu at (101.8, 68.5)
- added REF**: NPTH, NPTH, F.Cu at (78.0, 52.9)
- added REF**: NPTH, NPTH, F.Cu at (116.3, 69.5)
- added REF**: NPTH, NPTH, F.Cu at (132.0, 84.3)
- added REF**: NPTH, NPTH, F.Cu at (78.0, 90.0)
- added REF**: NPTH, NPTH, F.Cu at (125.3, 69.5)
- added REF**: NPTH, NPTH, F.Cu at (132.0, 44.8)
- added REF**: NPTH, NPTH, F.Cu at (102.6, 68.5)
- added REF**: NPTH, NPTH, F.Cu at (78.0, 77.8)
- added REF**: NPTH, NPTH, F.Cu at (132.0, 54.5)
- added REF**: NPTH, NPTH, F.Cu at (132.0, 56.9)
- added REF**: NPTH, NPTH, F.Cu at (86.4, 68.5)
- added REF**: NPTH, NPTH, F.Cu at (132.0, 26.2)
- added REF**: NPTH, NPTH, F.Cu at (84.7, 68.5)
- added REF**: NPTH, NPTH, F.Cu at (86.4, 69.5)
- added REF**: NPTH, NPTH, F.Cu at (78.0, 60.2)
- added REF**: NPTH, NPTH, F.Cu at (96.1, 68.5)
- added REF**: NPTH, NPTH, F.Cu at (106.6, 68.5)
- added REF**: NPTH, NPTH, F.Cu at (118.8, 68.5)
- added REF**: NPTH, NPTH, F.Cu at (118.8, 69.5)
- added REF**: NPTH, NPTH, F.Cu at (132.0, 106.1)
- added REF**: NPTH, NPTH, F.Cu at (132.0, 39.2)
- added REF**: NPTH, NPTH, F.Cu at (104.2, 68.5)
- added REF**: NPTH, NPTH, F.Cu at (132.0, 75.4)
- added REF**: NPTH, NPTH, F.Cu at (132.0, 33.5)
- added REF**: NPTH, NPTH, F.Cu at (98.5, 68.5)
- added REF**: NPTH, NPTH, F.Cu at (78.0, 28.7)
- added REF**: NPTH, NPTH, F.Cu at (132.0, 62.6)
- added REF**: NPTH, NPTH, F.Cu at (78.5, 68.0)
- added REF**: NPTH, NPTH, F.Cu at (132.0, 85.1)
- added REF**: NPTH, NPTH, F.Cu at (132.0, 100.5)
- added REF**: NPTH, NPTH, F.Cu at (132.0, 24.6)
- added REF**: NPTH, NPTH, F.Cu at (132.0, 90.0)
- added REF**: NPTH, NPTH, F.Cu at (128.6, 69.5)
- added REF**: NPTH, NPTH, F.Cu at (132.0, 89.2)
- added REF**: NPTH, NPTH, F.Cu at (132.0, 43.2)
- added REF**: NPTH, NPTH, F.Cu at (78.0, 94.0)
- added REF**: NPTH, NPTH, F.Cu at (132.0, 103.7)
- added REF**: NPTH, NPTH, F.Cu at (132.0, 96.4)
- added REF**: NPTH, NPTH, F.Cu at (95.3, 68.5)
- added REF**: NPTH, NPTH, F.Cu at (109.9, 69.5)
- added REF**: NPTH, NPTH, F.Cu at (132.0, 82.7)
- added REF**: NPTH, NPTH, F.Cu at (78.0, 106.1)
- added REF**: NPTH, NPTH, F.Cu at (115.5, 68.5)
- added REF**: NPTH, NPTH, F.Cu at (88.0, 69.5)
- added REF**: NPTH, NPTH, F.Cu at (132.0, 25.4)
- added REF**: NPTH, NPTH, F.Cu at (119.6, 68.5)
- added REF**: NPTH, NPTH, F.Cu at (131.5, 70.0)
- added REF**: NPTH, NPTH, F.Cu at (126.1, 69.5)
- added REF**: NPTH, NPTH, F.Cu at (132.0, 76.2)
- added REF**: NPTH, NPTH, F.Cu at (122.0, 68.5)
- added REF**: NPTH, NPTH, F.Cu at (89.6, 69.5)
- added REF**: NPTH, NPTH, F.Cu at (120.4, 68.5)
- added REF**: NPTH, NPTH, F.Cu at (83.1, 69.5)
- added REF**: NPTH, NPTH, F.Cu at (132.0, 60.2)
- added REF**: NPTH, NPTH, F.Cu at (132.0, 90.8)
- added REF**: NPTH, NPTH, F.Cu at (125.3, 68.5)
- added REF**: NPTH, NPTH, F.Cu at (88.0, 68.5)
- added REF**: NPTH, NPTH, F.Cu at (110.7, 68.5)
- added REF**: NPTH, NPTH, F.Cu at (78.0, 86.7)
- added REF**: NPTH, NPTH, F.Cu at (120.4, 69.5)
- added REF**: NPTH, NPTH, F.Cu at (78.0, 82.7)
- added REF**: NPTH, NPTH, F.Cu at (78.0, 56.1)
- added REF**: NPTH, NPTH, F.Cu at (122.8, 68.5)
- added REF**: NPTH, NPTH, F.Cu at (96.9, 68.5)
- added REF**: NPTH, NPTH, F.Cu at (132.0, 73.0)
- added REF**: NPTH, NPTH, F.Cu at (78.0, 64.2)
- added REF**: NPTH, NPTH, F.Cu at (78.0, 108.5)
- added REF**: NPTH, NPTH, F.Cu at (90.4, 69.5)
- added REF**: NPTH, NPTH, F.Cu at (132.0, 52.9)
- added REF**: NPTH, NPTH, F.Cu at (78.0, 96.4)
- added REF**: NPTH, NPTH, F.Cu at (78.0, 61.0)
- added REF**: NPTH, NPTH, F.Cu at (78.0, 42.4)
- added REF**: NPTH, NPTH, F.Cu at (78.0, 110.2)
- added REF**: NPTH, NPTH, F.Cu at (78.0, 90.8)
- added REF**: NPTH, NPTH, F.Cu at (78.0, 38.3)
- added REF**: NPTH, NPTH, F.Cu at (132.0, 95.6)
- added REF**: NPTH, NPTH, F.Cu at (78.0, 33.5)
- added REF**: NPTH, NPTH, F.Cu at (78.0, 57.7)
- added REF**: NPTH, NPTH, F.Cu at (132.0, 77.8)
- added REF**: NPTH, NPTH, F.Cu at (132.0, 87.5)
- added REF**: NPTH, NPTH, F.Cu at (78.0, 91.6)
- added REF**: NPTH, NPTH, F.Cu at (83.1, 68.5)
- added REF**: NPTH, NPTH, F.Cu at (132.0, 81.1)
- added REF**: NPTH, NPTH, F.Cu at (132.0, 98.8)
- added REF**: NPTH, NPTH, F.Cu at (78.0, 101.3)
- added REF**: NPTH, NPTH, F.Cu at (78.0, 98.8)
- added REF**: NPTH, NPTH, F.Cu at (78.0, 80.3)
- added REF**: NPTH, NPTH, F.Cu at (132.0, 47.2)
- added REF**: NPTH, NPTH, F.Cu at (78.0, 87.5)
- added REF**: NPTH, NPTH, F.Cu at (78.0, 93.2)
- added REF**: NPTH, NPTH, F.Cu at (132.0, 99.7)
- added REF**: NPTH, NPTH, F.Cu at (78.0, 97.2)
- added REF**: NPTH, NPTH, F.Cu at (78.0, 35.1)
- added REF**: NPTH, NPTH, F.Cu at (96.9, 69.5)
- added REF**: NPTH, NPTH, F.Cu at (110.7, 69.5)
- added REF**: NPTH, NPTH, F.Cu at (132.0, 31.1)
- added REF**: NPTH, NPTH, F.Cu at (132.0, 111.8)
- added REF**: NPTH, NPTH, F.Cu at (131.5, 68.0)
- added REF**: NPTH, NPTH, F.Cu at (78.0, 63.4)
- added REF**: NPTH, NPTH, F.Cu at (132.0, 78.7)
- added REF**: NPTH, NPTH, F.Cu at (124.4, 68.5)
- added REF**: NPTH, NPTH, F.Cu at (78.0, 83.5)
- added REF**: NPTH, NPTH, F.Cu at (132.0, 27.8)
- added REF**: NPTH, NPTH, F.Cu at (78.0, 52.1)
- added REF**: NPTH, NPTH, F.Cu at (132.0, 29.5)
- added REF**: NPTH, NPTH, F.Cu at (112.3, 68.5)
- added REF**: NPTH, NPTH, F.Cu at (132.0, 49.7)
- added REF**: NPTH, NPTH, F.Cu at (78.0, 107.7)
- added REF**: NPTH, NPTH, F.Cu at (85.6, 69.5)
- added REF**: NPTH, NPTH, F.Cu at (100.9, 69.5)
- added REF**: NPTH, NPTH, F.Cu at (121.2, 68.5)
- added REF**: NPTH, NPTH, F.Cu at (132.0, 110.2)
- added REF**: NPTH, NPTH, F.Cu at (117.2, 68.5)
- added REF**: NPTH, NPTH, F.Cu at (92.0, 68.5)
- added REF**: NPTH, NPTH, F.Cu at (132.0, 93.2)
- added REF**: NPTH, NPTH, F.Cu at (132.0, 72.9)
- added REF**: NPTH, NPTH, F.Cu at (88.8, 69.5)
- added REF**: NPTH, NPTH, F.Cu at (78.0, 78.7)
- added REF**: NPTH, NPTH, F.Cu at (132.0, 27.0)
- added REF**: NPTH, NPTH, F.Cu at (78.0, 30.3)
- added REF**: NPTH, NPTH, F.Cu at (118.0, 68.5)
- added REF**: NPTH, NPTH, F.Cu at (78.0, 111.8)
- added REF**: NPTH, NPTH, F.Cu at (78.0, 23.0)
- added REF**: NPTH, NPTH, F.Cu at (132.0, 97.2)
- added REF**: NPTH, NPTH, F.Cu at (78.0, 31.9)
- added REF**: NPTH, NPTH, F.Cu at (78.0, 62.6)
- added REF**: NPTH, NPTH, F.Cu at (93.7, 68.5)
- added REF**: NPTH, NPTH, F.Cu at (132.0, 77.0)
- added REF**: NPTH, NPTH, F.Cu at (132.0, 83.5)
- added REF**: NPTH, NPTH, F.Cu at (127.7, 68.5)
- added REF**: NPTH, NPTH, F.Cu at (78.0, 94.8)
- added REF**: NPTH, NPTH, F.Cu at (78.0, 95.6)
- added REF**: NPTH, NPTH, F.Cu at (132.0, 112.6)
- added REF**: NPTH, NPTH, F.Cu at (132.0, 81.9)
- added REF**: NPTH, NPTH, F.Cu at (78.0, 44.8)
- added REF**: NPTH, NPTH, F.Cu at (78.0, 23.8)
- added REF**: NPTH, NPTH, F.Cu at (126.1, 68.5)
- added REF**: NPTH, NPTH, F.Cu at (112.3, 69.5)
- added REF**: NPTH, NPTH, F.Cu at (92.8, 68.5)
- added REF**: NPTH, NPTH, F.Cu at (90.4, 68.5)
- added REF**: NPTH, NPTH, F.Cu at (78.5, 69.0)
- added REF**: NPTH, NPTH, F.Cu at (132.0, 23.0)
- added REF**: NPTH, NPTH, F.Cu at (105.8, 68.5)
- added REF**: NPTH, NPTH, F.Cu at (132.0, 91.6)
- added REF**: NPTH, NPTH, F.Cu at (93.7, 69.5)
- added REF**: NPTH, NPTH, F.Cu at (78.0, 48.0)
- added REF**: NPTH, NPTH, F.Cu at (132.0, 79.5)
- added REF**: NPTH, NPTH, F.Cu at (123.6, 69.5)
- added REF**: NPTH, NPTH, F.Cu at (78.0, 114.2)
- added REF**: NPTH, NPTH, F.Cu at (113.1, 69.5)
- added REF**: NPTH, NPTH, F.Cu at (101.8, 69.5)
- added REF**: NPTH, NPTH, F.Cu at (132.0, 40.8)
- added REF**: NPTH, NPTH, F.Cu at (94.5, 68.5)
- added REF**: NPTH, NPTH, F.Cu at (78.0, 53.7)
- added REF**: NPTH, NPTH, F.Cu at (95.3, 69.5)
- added REF**: NPTH, NPTH, F.Cu at (132.0, 22.9)
- added REF**: NPTH, NPTH, F.Cu at (122.8, 69.5)
- added REF**: NPTH, NPTH, F.Cu at (82.3, 68.5)
- added REF**: NPTH, NPTH, F.Cu at (91.2, 69.5)
- added REF**: NPTH, NPTH, F.Cu at (132.0, 106.9)
- added REF**: NPTH, NPTH, F.Cu at (78.0, 102.9)
- added REF**: NPTH, NPTH, F.Cu at (78.0, 26.2)
- added REF**: NPTH, NPTH, F.Cu at (78.0, 35.9)
- added REF**: NPTH, NPTH, F.Cu at (78.0, 44.0)
- added REF**: NPTH, NPTH, F.Cu at (85.6, 68.5)
- added REF**: NPTH, NPTH, F.Cu at (132.0, 107.7)
- added REF**: NPTH, NPTH, F.Cu at (78.0, 48.8)
- added REF**: NPTH, NPTH, F.Cu at (96.1, 69.5)
- added REF**: NPTH, NPTH, F.Cu at (78.0, 73.0)
- added REF**: NPTH, NPTH, F.Cu at (132.0, 101.3)
- added REF**: NPTH, NPTH, F.Cu at (114.7, 68.5)
- added REF**: NPTH, NPTH, F.Cu at (87.2, 68.5)
- added REF**: NPTH, NPTH, F.Cu at (132.0, 23.8)
- added REF**: NPTH, NPTH, F.Cu at (132.0, 37.5)
- added REF**: NPTH, NPTH, F.Cu at (132.0, 92.4)
- added REF**: NPTH, NPTH, F.Cu at (84.7, 69.5)
- added REF**: NPTH, NPTH, F.Cu at (126.9, 68.5)
- added REF**: NPTH, NPTH, F.Cu at (78.0, 27.0)
- added REF**: NPTH, NPTH, F.Cu at (108.2, 69.5)
- added REF**: NPTH, NPTH, F.Cu at (132.0, 114.2)
- added REF**: NPTH, NPTH, F.Cu at (121.2, 69.5)
- added REF**: NPTH, NPTH, F.Cu at (78.0, 72.9)
- added REF**: NPTH, NPTH, F.Cu at (94.5, 69.5)
- added REF**: NPTH, NPTH, F.Cu at (78.0, 47.2)
- added REF**: NPTH, NPTH, F.Cu at (109.9, 68.5)
- added REF**: NPTH, NPTH, F.Cu at (104.2, 69.5)
- added REF**: NPTH, NPTH, F.Cu at (108.2, 68.5)
- added REF**: NPTH, NPTH, F.Cu at (78.0, 111.0)
- added REF**: NPTH, NPTH, F.Cu at (83.9, 68.5)
- added REF**: NPTH, NPTH, F.Cu at (132.0, 73.8)
- added REF**: NPTH, NPTH, F.Cu at (78.0, 77.0)
- added REF**: NPTH, NPTH, F.Cu at (78.0, 32.7)
- added REF**: NPTH, NPTH, F.Cu at (87.2, 69.5)
- added REF**: NPTH, NPTH, F.Cu at (116.3, 68.5)
- added REF**: NPTH, NPTH, F.Cu at (132.0, 44.0)
- added REF**: NPTH, NPTH, F.Cu at (132.0, 46.4)
- added REF**: NPTH, NPTH, F.Cu at (92.8, 69.5)
- added REF**: NPTH, NPTH, F.Cu at (126.9, 69.5)
- added REF**: NPTH, NPTH, F.Cu at (132.0, 64.2)
- added REF**: NPTH, NPTH, F.Cu at (103.4, 68.5)
- added REF**: NPTH, NPTH, F.Cu at (78.0, 55.3)
- added REF**: NPTH, NPTH, F.Cu at (113.1, 68.5)
- added REF**: NPTH, NPTH, F.Cu at (98.5, 69.5)
- added REF**: NPTH, NPTH, F.Cu at (128.5, 69.5)
- added REF**: NPTH, NPTH, F.Cu at (78.0, 46.4)
- added REF**: NPTH, NPTH, F.Cu at (78.0, 75.4)
- added REF**: NPTH, NPTH, F.Cu at (78.0, 105.3)
- added REF**: NPTH, NPTH, F.Cu at (78.0, 22.9)
- added REF**: NPTH, NPTH, F.Cu at (105.8, 69.5)
- added REF**: NPTH, NPTH, F.Cu at (78.0, 81.1)
- added REF**: NPTH, NPTH, F.Cu at (78.0, 29.5)
- added REF**: NPTH, NPTH, F.Cu at (107.4, 69.5)
- added REF**: NPTH, NPTH, F.Cu at (78.0, 51.3)
- added REF**: NPTH, NPTH, F.Cu at (78.0, 106.9)
- added REF**: NPTH, NPTH, F.Cu at (99.3, 69.5)
- added REF**: NPTH, NPTH, F.Cu at (124.4, 69.5)
- added REF**: NPTH, NPTH, F.Cu at (132.0, 109.3)
- added REF**: NPTH, NPTH, F.Cu at (132.0, 61.8)
- added REF**: NPTH, NPTH, F.Cu at (78.0, 81.9)
- added REF**: NPTH, NPTH, F.Cu at (81.5, 68.5)
- added REF**: NPTH, NPTH, F.Cu at (132.0, 80.3)
- added REF**: NPTH, NPTH, F.Cu at (88.8, 68.5)
- added REF**: NPTH, NPTH, F.Cu at (107.4, 68.5)
- added REF**: NPTH, NPTH, F.Cu at (78.0, 45.6)
- added REF**: NPTH, NPTH, F.Cu at (78.0, 41.6)
- added REF**: NPTH, NPTH, F.Cu at (132.0, 55.3)
- added REF**: NPTH, NPTH, F.Cu at (113.9, 69.5)
- added REF**: NPTH, NPTH, F.Cu at (78.0, 79.5)
- added REF**: NPTH, NPTH, F.Cu at (78.0, 40.8)
- added REF**: NPTH, NPTH, F.Cu at (128.6, 68.5)
- added REF**: NPTH, NPTH, F.Cu at (132.0, 94.0)
- added REF**: NPTH, NPTH, F.Cu at (132.0, 108.5)
- added REF**: NPTH, NPTH, F.Cu at (81.5, 69.5)
- added REF**: NPTH, NPTH, F.Cu at (132.0, 48.0)
- added REF**: NPTH, NPTH, F.Cu at (132.0, 111.0)
- added REF**: NPTH, NPTH, F.Cu at (78.0, 76.2)
- added REF**: NPTH, NPTH, F.Cu at (132.0, 30.3)
- added REF**: NPTH, NPTH, F.Cu at (78.0, 50.5)
- added REF**: NPTH, NPTH, F.Cu at (99.3, 68.5)
- added REF**: NPTH, NPTH, F.Cu at (78.0, 115.0)
- added REF**: NPTH, NPTH, F.Cu at (78.0, 100.5)
- added REF**: NPTH, NPTH, F.Cu at (102.6, 69.5)
- added REF**: NPTH, NPTH, F.Cu at (78.0, 113.4)
- added REF**: NPTH, NPTH, F.Cu at (78.0, 98.0)
- added REF**: NPTH, NPTH, F.Cu at (78.0, 37.5)
- added REF**: NPTH, NPTH, F.Cu at (114.7, 69.5)
- added REF**: NPTH, NPTH, F.Cu at (106.6, 69.5)
- added REF**: NPTH, NPTH, F.Cu at (132.0, 32.7)
- added REF**: NPTH, NPTH, F.Cu at (82.3, 69.5)
- added REF**: NPTH, NPTH, F.Cu at (132.0, 104.5)
- added REF**: NPTH, NPTH, F.Cu at (100.1, 68.5)
- added REF**: NPTH, NPTH, F.Cu at (132.0, 85.9)
- added REF**: NPTH, NPTH, F.Cu at (132.0, 48.8)
- added REF**: NPTH, NPTH, F.Cu at (78.0, 85.1)
- added REF**: NPTH, NPTH, F.Cu at (100.9, 68.5)
- added REF**: NPTH, NPTH, F.Cu at (132.0, 28.7)
- added REF**: NPTH, NPTH, F.Cu at (78.0, 104.5)
- added REF**: NPTH, NPTH, F.Cu at (92.0, 69.5)
- added REF**: NPTH, NPTH, F.Cu at (113.9, 68.5)
- added REF**: NPTH, NPTH, F.Cu at (78.0, 61.8)
- added REF**: NPTH, NPTH, F.Cu at (100.1, 69.5)
- added REF**: NPTH, NPTH, F.Cu at (132.0, 63.4)
- added REF**: NPTH, NPTH, F.Cu at (132.0, 98.0)
- added REF**: NPTH, NPTH, F.Cu at (132.0, 34.3)
- added REF**: NPTH, NPTH, F.Cu at (78.0, 65.0)
- added REF**: NPTH, NPTH, F.Cu at (78.0, 85.9)
- added REF**: NPTH, NPTH, F.Cu at (132.0, 94.8)
- added REF**: NPTH, NPTH, F.Cu at (78.0, 31.1)
- added REF**: NPTH, NPTH, F.Cu at (132.0, 105.3)
- added REF**: NPTH, NPTH, F.Cu at (78.0, 112.6)
- added REF**: NPTH, NPTH, F.Cu at (132.0, 35.1)
- added REF**: NPTH, NPTH, F.Cu at (115.5, 69.5)
- added REF**: NPTH, NPTH, F.Cu at (117.2, 69.5)
- added REF**: NPTH, NPTH, F.Cu at (78.0, 109.3)
- added REF**: NPTH, NPTH, F.Cu at (132.0, 58.5)
- added REF**: NPTH, NPTH, F.Cu at (78.0, 92.4)
- added REF**: NPTH, NPTH, F.Cu at (105.0, 68.5)
- added REF**: NPTH, NPTH, F.Cu at (78.0, 34.3)
- added REF**: NPTH, NPTH, F.Cu at (132.0, 52.1)
- added REF**: NPTH, NPTH, F.Cu at (111.5, 68.5)
- added REF**: NPTH, NPTH, F.Cu at (78.0, 73.8)
- added REF**: NPTH, NPTH, F.Cu at (78.0, 103.7)
- added REF**: NPTH, NPTH, F.Cu at (78.0, 39.2)
- added REF**: NPTH, NPTH, F.Cu at (78.0, 40.0)
- added REF**: NPTH, NPTH, F.Cu at (132.0, 113.4)
- added REF**: NPTH, NPTH, F.Cu at (119.6, 69.5)
- added REF**: NPTH, NPTH, F.Cu at (109.1, 69.5)
- added REF**: NPTH, NPTH, F.Cu at (131.5, 69.0)
- added REF**: NPTH, NPTH, F.Cu at (132.0, 56.1)
- added REF**: NPTH, NPTH, F.Cu at (105.0, 69.5)
- added REF**: NPTH, NPTH, F.Cu at (132.0, 40.0)
- added REF**: NPTH, NPTH, F.Cu at (123.6, 68.5)
- added REF**: NPTH, NPTH, F.Cu at (83.9, 69.5)
- added REF**: NPTH, NPTH, F.Cu at (132.0, 51.3)
- added REF**: NPTH, NPTH, F.Cu at (78.0, 25.4)
- added REF**: NPTH, NPTH, F.Cu at (132.0, 53.7)
- added REF**: NPTH, NPTH, F.Cu at (132.0, 31.9)
- added REF**: NPTH, NPTH, F.Cu at (78.0, 54.5)
- added REF**: NPTH, NPTH, F.Cu at (132.0, 35.9)
- added REF**: NPTH, NPTH, F.Cu at (132.0, 74.6)
- added REF**: NPTH, NPTH, F.Cu at (78.0, 58.5)
- added REF**: NPTH, NPTH, F.Cu at (109.1, 68.5)
- added REF**: NPTH, NPTH, F.Cu at (78.0, 99.7)
- added REF**: NPTH, NPTH, F.Cu at (78.0, 24.6)
- added REF**: NPTH, NPTH, F.Cu at (78.0, 36.7)
- added REF**: NPTH, NPTH, F.Cu at (97.7, 69.5)
- added REF**: NPTH, NPTH, F.Cu at (132.0, 59.3)
- added REF**: NPTH, NPTH, F.Cu at (132.0, 61.0)
- added REF**: NPTH, NPTH, F.Cu at (132.0, 65.0)
- added REF**: NPTH, NPTH, F.Cu at (132.0, 57.7)
- added REF**: NPTH, NPTH, F.Cu at (103.4, 69.5)
- added REF**: NPTH, NPTH, F.Cu at (78.0, 49.7)
- added REF**: NPTH, NPTH, F.Cu at (118.0, 69.5)
- added REF**: NPTH, NPTH, F.Cu at (132.0, 38.3)
- added REF**: NPTH, NPTH, F.Cu at (78.0, 84.3)
- added REF**: NPTH, NPTH, F.Cu at (89.6, 68.5)
- added REF**: NPTH, NPTH, F.Cu at (132.0, 36.7)
- added REF**: NPTH, NPTH, F.Cu at (132.0, 115.0)
- added REF**: NPTH, NPTH, F.Cu at (132.0, 42.4)
- added REF**: NPTH, NPTH, F.Cu at (132.0, 102.1)
- added REF**: NPTH, NPTH, F.Cu at (132.0, 50.5)
- added REF**: NPTH, NPTH, F.Cu at (132.0, 45.6)
- added REF**: NPTH, NPTH, F.Cu at (78.5, 70.0)
- added REF**: NPTH, NPTH, F.Cu at (132.0, 88.3)
- added TP1: 3V3, TestPoint:TestPoint_Pad_D1.0mm, B.Cu at (108.8, 29.0)
- added TP1: 3V3, TestPoint:TestPoint_Pad_D1.0mm, B.Cu at (108.8, 79.0)
- added TP3: SWDIO, TestPoint:TestPoint_Pad_D1.0mm, B.Cu at (108.8, 27.7)
- added TP3: SWDIO, TestPoint:TestPoint_Pad_D1.0mm, B.Cu at (108.8, 77.7)
- added TP4: SWCLK, TestPoint:TestPoint_Pad_D1.0mm, B.Cu at (108.8, 76.4)
- added TP4: SWCLK, TestPoint:TestPoint_Pad_D1.0mm, B.Cu at (108.8, 26.4)
- added TP5: GND, TestPoint:TestPoint_Pad_D1.0mm, B.Cu at (108.8, 75.2)
- added TP5: GND, TestPoint:TestPoint_Pad_D1.0mm, B.Cu at (108.8, 25.2)
- added U1: AZ1117-3.3, Package_TO_SOT_SMD:SOT-223-3_TabPin2, F.Cu at (100.4, 52.1)
- added U1: AZ1117-3.3, Package_TO_SOT_SMD:SOT-223-3_TabPin2, F.Cu at (100.4, 102.1)
- added U2: MP2315, Package_TO_SOT_SMD:TSOT-23-8, B.Cu at (100.0, 106.7)
- added U2: MP2315, Package_TO_SOT_SMD:TSOT-23-8, B.Cu at (100.0, 56.7)
- added kibuzzard-63CD1E61: G***, kibuzzard-63CD1E61, B.Cu at (110.7, 79.0)
- added kibuzzard-63CD1E61: G***, kibuzzard-63CD1E61, B.Cu at (110.7, 29.0)
- added kibuzzard-63CD1E7F: G***, kibuzzard-63CD1E7F, B.Cu at (110.7, 25.1)
- added kibuzzard-63CD1E7F: G***, kibuzzard-63CD1E7F, B.Cu at (110.7, 75.1)
- added kibuzzard-63CD1EC0: G***, kibuzzard-63CD1EC0, B.Cu at (110.7, 76.4)
- added kibuzzard-63CD1EC0: G***, kibuzzard-63CD1EC0, B.Cu at (110.7, 26.4)
- added kibuzzard-63CD1EC5: G***, kibuzzard-63CD1EC5, B.Cu at (110.7, 27.7)
- added kibuzzard-63CD1EC5: G***, kibuzzard-63CD1EC5, B.Cu at (110.7, 77.7)
- L2 (x2): value NC -> 22u
- R12 (x2): value NC -> 22
- moved C10 2.00 mm to (104.2, 107.0)
- moved C11 2.00 mm to (121.0, 89.0)
- moved C12 2.00 mm to (107.0, 103.6)
- moved C13 2.00 mm to (123.5, 86.5)
- moved C14 2.00 mm to (126.7, 81.9)
- moved C15 2.00 mm to (87.9, 115.4)
- moved C16 2.00 mm to (115.9, 79.2)
- moved C18 2.00 mm to (100.3, 101.4)
- moved C22 2.00 mm to (86.8, 79.2)
- moved C23 2.00 mm to (80.6, 79.0)
- moved C24 2.00 mm to (85.3, 76.3)
- moved C3 2.00 mm to (106.1, 86.9)
- moved C6 2.00 mm to (100.8, 107.0)
- moved C9 2.00 mm to (123.5, 89.8)
- moved D2 2.00 mm to (115.7, 110.2)
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Connections:
- U8 pad 27: Board_0-unconnected-(U8-Pad27) -> Board_0-IO0
- U8 pad 27: Board_1-unconnected-(U8-Pad27) -> Board_1-IO0
Routing:
- net Board_0-Net-(C1-Pad1): track 21.0 -> 67.4 mm, vias 1 -> 3
- net Board_1-Net-(C1-Pad1): track 21.0 -> 67.4 mm, vias 1 -> 3
- net Board_0-IO0: track 0.00 -> 44.2 mm, vias 0 -> 1
- net Board_1-IO0: track 0.00 -> 44.2 mm, vias 0 -> 1
- net Board_1-+BATT: track 65.6 -> 76.7 mm, vias 2 -> 5
- net Board_0-+BATT: track 65.6 -> 76.7 mm, vias 2 -> 5
- net Board_0-GND: track 52.5 -> 43.3 mm, vias 44 -> 94
- net Board_1-GND: track 52.5 -> 43.3 mm, vias 44 -> 94
- net Board_0-Net-(R8-Pad1): track 10.6 -> 2.08 mm, vias 2 -> 0
- net Board_1-Net-(R8-Pad1): track 10.6 -> 2.08 mm, vias 2 -> 0
- net Board_1-Net-(R9-Pad1): track 10.5 -> 2.42 mm, vias 2 -> 0
- net Board_0-Net-(R9-Pad1): track 10.5 -> 2.42 mm, vias 2 -> 0
- net Board_0-+5V: track 145.0 -> 138.4 mm
- net Board_1-+5V: track 145.0 -> 138.4 mm
- net Board_1-+3V3: track 206.7 -> 211.1 mm
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Other:
- board size 73 x 102 mm -> 67 x 98 mm
- board text added: "BSD-3-Clause open source hardware By @wilicw"
- board text added: "NCKU ISP Avionics ISP32 v2.1"
- board text removed: "48mm x 53mm M3 Screw Input 5V~16V By @wilicw"
- board text removed: "BSD-3-Clause open source hardware"
- board text removed: "NCKU ISP Avionics ISP32 v2"
- board text removed: "V-CUT"
